File: pcb/ai_candle.brd (EAGLE design)
At the start: 27.9 x 27.9 mm, 6 parts, among them J1 JST-2-MALE

Commit message: updating
Routing:
- net GND: track 28.0 -> 29.3 mm
- net N$2: track 22.5 -> 21.5 mm
Changed lines of the file:
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@@
 <contactref element="BATT" pad="3"/>
 <contactref element="J1" pad="2"/>
-<wire x1="13.97" y1="22.765" x2="13.97" y2="10.16" width="0.4064" layer="1"/>
+<wire x1="13.97" y1="23.495" x2="13.97" y2="10.16" width="0.4064" layer="1"/>
 <wire x1="12.97" y1="7.764" x2="12.97" y2="21.511" width="0.4064" layer="16"/>
-<wire x1="12.97" y1="21.511" x2="13.97" y2="22.765" width="0.4064" layer="16"/>
+<wire x1="12.97" y1="21.511" x2="13.97" y2="23.495" width="0.4064" layer="16"/>
 <polygon width="0.254" layer="16">
 <vertex x="0" y="0"/>
@@
 <contactref element="LED2" pad="C"/>
 <contactref element="SW1" pad="1"/>
-<wire x1="13.97" y1="26.765" x2="19.897975" y2="20.583025" width="0.4064" layer="1"/>
+<wire x1="13.97" y1="26.035" x2="19.897975" y2="20.583025" width="0.4064" layer="1"/>
 <wire x1="19.897975" y1="20.583025" x2="22.596971875" y2="20.583025" width="0.4064" layer="1"/>
-<wire x1="13.97" y1="26.765" x2="8.042025" y2="20.583025" width="0.4064" layer="1"/>
+<wire x1="13.97" y1="26.035" x2="8.042025" y2="20.583025" width="0.4064" layer="1"/>
 <wire x1="8.042025" y1="20.583025" x2="5.343025" y2="20.583025" width="0.4064" layer="1"/>
 </signal>
